Commit message: Robot Final Model + ROS2 control + Gripper Control

File: mam_eurobot_2026/urdf/four_wheel_robot.xacro (robot description, xacro)
@@ -4,14 +4,22 @@
 <!-- karamdali93@gmail.com -->
 <!-- This is a simple 4 mecanume wheels robot with a tow figer gripper in the front of it -->
-<!-- P.S : Any change in the robot dimentions should be reflected in config/mecanum_drive_controller.yaml -->
+<!-- P.S  Any change in the robot dimentions should be reflected in config/mecanum_drive_controller . yaml -->
 <!-- Robot Dimensions Parameters -->
-<xacro:property name="robot_x" value="0.28" /> <!-- Chassis length -->
-<xacro:property name="robot_y" value="0.22" /> <!-- Chassis width -->
-<xacro:property name="robot_z" value="0.05" /> <!-- Chassis height (thickness) -->
-<xacro:property name="chassis_mass" value="0.75" />
-<!-- Chassis Inertia Parameters -->
-<xacro:property name="ixx" value="${0.001191615 * chassis_mass}" />
-<xacro:property name="iyy" value="${0.004051490 * chassis_mass}" />
-<xacro:property name="izz" value="${0.004766458 * chassis_mass}" />
+<xacro:property name="robot_x" value="0.28" /> <!-- base_link length -->
+<xacro:property name="robot_y" value="0.22" /> <!-- base_link width -->
+<xacro:property name="robot_z" value="0.05" /> <!-- base_link height (thickness) -->
+<xacro:property name="base_link_mass" value="0.75" />
+<!-- base_link Inertia Parameters -->
+<xacro:property name="base_link_ixx" value="${base_link_mass/12 * (robot_y*robot_y + robot_z*robot_z)}" />
+<xacro:property name="base_link_iyy" value="${base_link_mass/12 * (robot_x*robot_x + robot_z*robot_z)}" />
+<xacro:property name="base_link_izz" value="${base_link_mass/12 * (robot_x*robot_x + robot_y*robot_y)}" />
+<!-- Robot AruCo Parameters -->
+<xacro:property name="aruco_dimenstion" value="0.1" />
+<xacro:property name="aruco_thick" value="0.002" />
+<xacro:property name="aruco_mass" value="0.01" />
+<xacro:property name="aruco_ixx" value="${aruco_mass/12 * (aruco_dimenstion*aruco_dimenstion + aruco_thick*aruco_thick)}" />
+<xacro:property name="aruco_iyy" value="${aruco_mass/12 * (aruco_dimenstion*aruco_dimenstion + aruco_thick*aruco_thick)}" />
+<xacro:property name="aruco_izz" value="${aruco_mass/12 * (aruco_dimenstion*aruco_dimenstion + aruco_dimenstion*aruco_dimenstion)}" />
+<xacro:property name="aruco_z_offset" value="${base_link_center_z+robot_z/2 + 0.001}" />
 <!-- Wheel Parameters -->
 <xacro:property name="wheel_radius" value="0.03" />
@@ -22,8 +30,8 @@
 <xacro:property name="wheel_iyy" value="${(1.0/12.0) * wheel_mass * (3*wheel_radius*wheel_radius + wheel_width*wheel_width)}" />
 <xacro:property name="wheel_izz" value="${wheel_iyy}" />
-<!-- We place the CHASSIS center higher so the wheels touch ground at z=0. -->
-<!-- chassis_center_z = wheel_radius + robot_z/2 -->
-<xacro:property name="chassis_center_z" value="${wheel_radius + (robot_z/2)}" />
-<!-- Calculated Joint Positions (relative to CHASSIS origin) -->
+<!-- We place the base_link center higher so the wheels touch ground at z=0. -->
+<!-- base_link_center_z = wheel_radius + robot_z/2 -->
+<xacro:property name="base_link_center_z" value="${wheel_radius + (robot_z/2)}" />
+<!-- Calculated Joint Positions (relative to base_link origin) -->
 <xacro:property name="front_x" value="${(robot_x / 2) - wheel_radius}" />
 <xacro:property name="rear_x" value="${(-robot_x / 2) + wheel_radius}" />
@@ -31,5 +39,5 @@
 <xacro:property name="right_y" value="${(-robot_y / 2) - (wheel_width / 2)}" />
 <!-- joint z is set so wheel center absolute z == wheel_radius (wheel touches ground) -->
-<!-- joint z relative to chassis origin = -robot_z/2 -->
+<!-- joint z relative to base_link origin = -robot_z/2 -->
 <xacro:property name="wheel_joint_z" value="${robot_z/2}"/>
 <!-- Gripper specifications -->
@@ -41,21 +49,21 @@
 <xacro:property name="gripper_L_y_location" value="${((robot_y / 2) - (gripper_y/2))}" />
 <xacro:property name="gripper_R_y_location" value="${-((robot_y / 2) - (gripper_y/2))}" />
-<xacro:property name="gripper_z_location" value="${chassis_center_z/2}" />
+<xacro:property name="gripper_z_location" value="${base_link_center_z/2}" />
 <!-- Crate length -->
 <xacro:property name="crate_length" value="0.15" />
-<!-- Base chassis -->
-<link name="chassis">
+<!-- Base base_link -->
+<link name="base_link">
   <inertial>
-    <mass value="${chassis_mass}"/>
+    <mass value="${base_link_mass}"/>
     <inertia
-    ixx="${ixx}"
+    ixx="${base_link_ixx}"
     ixy="0.0"
     ixz="0.0"
-    iyy="${iyy}"
+    iyy="${base_link_iyy}"
     iyz="0.0"
-    izz="${izz}"/>
+    izz="${base_link_izz}"/>
     </inertial>
   <visual>
-    <origin rpy="0 0 0" xyz="0 0 ${chassis_center_z}"/>
+    <origin rpy="0 0 0" xyz="0 0 ${base_link_center_z}"/>
     <geometry>
       <box size="${robot_x} ${robot_y} ${robot_z}"/>
@@ -66,5 +74,5 @@
   </visual>
   <collision>
-    <origin rpy="0 0 0" xyz="0 0 ${chassis_center_z}"/>
+    <origin rpy="0 0 0" xyz="0 0 ${base_link_center_z}"/>
     <geometry>
       <box size="${robot_x} ${robot_y} ${robot_z}"/>
@@ -72,4 +80,48 @@
   </collision>
 </link>
+<!-- Robot AruCo  -->
+<link name="aruco">
+  <inertial>
+    <mass value="${aruco_mass}"/>
+    <inertia
+      ixx="${aruco_ixx}"
+      ixy="0.0"
+      ixz="0.0"
+      iyy="${aruco_iyy}"
+      iyz="0.0"
+      izz="${aruco_izz}"/>
+  </inertial>
+  <!-- Main ArUCo body (white) -->
+  <visual>
+    <origin rpy="0 0 1.57079" xyz="0 0 0"/>
+    <geometry>
+      <box size="${aruco_dimenstion} ${aruco_dimenstion} ${aruco_thick}"/>
+    </geometry>
+    <material name="white">
+      <color rgba="1.0 1.0 1.0 1"/>
+    </material>
+  </visual>
+  <!-- ArUCo texture on top surface -->
+  <visual name="aruco_top">
+    <origin xyz="0 0 ${aruco_thick/2}" rpy="0 0 0"/>
+    <geometry>
+      <box size="${aruco_dimenstion} ${aruco_dimenstion} 0.001"/>
+    </geometry>
+    <material name="white">
+      <color rgba="1 1 1 0"/>
+    </material>
+  </visual>
+  <collision>
+    <origin rpy="0 0 0" xyz="0 0 0"/>
+    <geometry>
+      <box size="${aruco_dimenstion} ${aruco_dimenstion} ${aruco_thick}"/>
+    </geometry>
+  </collision>
+</link>
+<joint name="aruco_joint" type="fixed">
+  <parent link="base_link"/>
+  <child link="aruco"/>
+  <origin xyz="0 0 ${aruco_z_offset}" rpy="0 0 0"/>
+</joint>
 <!-- Gripper Macro -->
 <xacro:macro name="gripper" params="name x y z">
@@ -123,8 +175,8 @@
 </xacro:macro>
 <!-- Creat the gripper joints -->
-<xacro:gripper_joint name="gripper_L_joint" parent="chassis" child="gripper_L"
+<xacro:gripper_joint name="gripper_L_joint" parent="base_link" child="gripper_L"
 x="${gripper_x_location}" y="${gripper_L_y_location}" z="${gripper_z_location}"
 robot_dimention_y="${robot_y}" side="left"/>
-<xacro:gripper_joint name="gripper_R_joint" parent="chassis" child="gripper_R"
+<xacro:gripper_joint name="gripper_R_joint" parent="base_link" child="gripper_R"
 x="${gripper_x_location}" y="${gripper_R_y_location}" z="${gripper_z_location}"
 robot_dimention_y="${robot_y}" side="right"/>
@@ -180,11 +232,11 @@
 </xacro:macro>
 <!-- Create Wheel Joints -->
-<xacro:wheel_joint name="front_left_wheel_joint" parent="chassis" child="front_left_wheel"
+<xacro:wheel_joint name="front_left_wheel_joint" parent="base_link" child="front_left_wheel"
 x="${front_x}" y="${left_y}" z="${wheel_joint_z}"/>
-<xacro:wheel_joint name="front_right_wheel_joint" parent="chassis" child="front_right_wheel"
+<xacro:wheel_joint name="front_right_wheel_joint" parent="base_link" child="front_right_wheel"
 x="${front_x}" y="${right_y}" z="${wheel_joint_z}"/>
-<xacro:wheel_joint name="rear_left_wheel_joint" parent="chassis" child="rear_left_wheel"
+<xacro:wheel_joint name="rear_left_wheel_joint" parent="base_link" child="rear_left_wheel"
 x="${rear_x}" y="${left_y}" z="${wheel_joint_z}"/>
-<xacro:wheel_joint name="rear_right_wheel_joint" parent="chassis" child="rear_right_wheel"
+<xacro:wheel_joint name="rear_right_wheel_joint" parent="base_link" child="rear_right_wheel"
 x="${rear_x}" y="${right_y}" z="${wheel_joint_z}"/>
 <!-- Gazebo extension used to emulate mecanum wheel frictions -->
@@ -195,8 +247,8 @@
         <friction>
           <ode>
-            <mu>2.0</mu>
+            <mu>1.0</mu>
             <mu2>0.0</mu2>
-            <!-- We express friction direction in CHASSIS frame to avoid confusion -->
-            <fdir1 ignition:expressed_in="chassis">${value}</fdir1>
+            <!-- We express friction direction in base_link frame to avoid confusion -->
+            <fdir1 ignition:expressed_in="base_link">${value}</fdir1>
           </ode>
         </friction>
@@ -205,5 +257,5 @@
   </gazebo>
 </xacro:macro>
-<!-- Chassis-frame mecanum directions (X forward, Y left) -->
+<!-- base_link-frame mecanum directions (X forward, Y left) -->
 <xacro:gazebo name="front_left_wheel"  value="1 -1 0"/>
 <xacro:gazebo name="front_right_wheel" value="1 1 0"/>
@@ -255,4 +307,21 @@
   </joint>
 </ros2_control>
+<!-- IMU sensor -->
+<link name="imu_link">
+  <visual>
+    <geometry>
+      <box size="0.02 0.02 0.01"/>
+    </geometry>
+  </visual>
+  <inertial>
+    <mass value="0.01"/>
+    <inertia ixx="1e-5" ixy="0" ixz="0" iyy="1e-5" iyz="0" izz="1e-5"/>
+  </inertial>
+</link>
+<joint name="imu_joint" type="fixed">
+  <parent link="base_link"/>
+  <child link="imu_link"/>
+  <origin xyz="0 0 0.05" rpy="0 0 0"/>
+</joint>
 <!-- ROS2 Control plugin and topic re-mapping -->
 <gazebo>
@@ -265,3 +334,33 @@
   </plugin>
 </gazebo>
+<gazebo reference="aruco">
+  <visual name="aruco_top">
+    <material>
+      <diffuse>1 1 1 1</diffuse>
+      <pbr>
+        <metal>
+          <albedo_map>
+            model://models/aruco/aruco_17.png
+          </albedo_map>
+          <metalness>0.0</metalness>
+          <roughness>0.0</roughness>
+        </metal>
+      </pbr>
+      <double_sided>true</double_sided>
+    </material>
+  </visual>
+</gazebo>
+<gazebo reference="imu_link">
+  <sensor name="imu_sensor" type="imu">
+    <topic>imu</topic>
+    <always_on>true</always_on>
+    <update_rate>25</update_rate>
+    <visualize>true</visualize>
+    <gz_frame_id>imu_link</gz_frame_id>
+    <plugin
+      filename="gz-sim-imu-system"
+      name="gz::sim::systems::Imu">
+    </plugin>
+  </sensor>
+</gazebo>
 </robot>

Commit message: Final working NAV2 stack

File: mam_eurobot_2026/urdf/four_wheel_robot.xacro (robot description, xacro)
@@ -166,9 +166,9 @@
     <xacro:if value="${side == 'left'}">
       <axis xyz="0 -1 0"/>
-      <limit lower="0" upper="${(robot_dimention_y - (crate_length + 2*gripper_y)) / 2}" effort="1000" velocity="0.1"/>
+      <limit lower="0" upper="${((robot_dimention_y - (crate_length + 2*gripper_y)) / 2)+0.01}" effort="1000" velocity="0.1"/>
     </xacro:if>
     <xacro:if value="${side == 'right'}">
       <axis xyz="0 1 0"/>
-      <limit lower="0" upper="${(robot_dimention_y - (crate_length + 2*gripper_y)) / 2}" effort="1000" velocity="0.1"/>
+      <limit lower="0" upper="${((robot_dimention_y - (crate_length + 2*gripper_y)) / 2)+0.01}" effort="1000" velocity="0.1"/>
     </xacro:if>
   </joint>
